File: hw/sch_pcb/SIPM02.kicad_sch (KiCad schematic)
At the start: 39 parts, among them J1 HEADER_2x01_PARALLEL, J10 HEADER_2x01_PARALLEL, J2 HEADER_2x01_PARALLEL, J3 HEADER_2x01_PARALLEL, J4 HEADER_2x01_PARALLEL, J5 HEADER_2x01_PARALLEL, J6 HEADER_2x01_PARALLEL, J7 HEADER_2x01_PARALLEL, J8 HEADER_2x01_PARALLEL, J9 HEADER_2x01_PARALLEL, M1 HOLE, M2 HOLE, M3 HOLE, M4 HOLE, U1 MICROFC-60035-SMT-TR(1), U2 OPA836IDB

Commit message: Cleanup renaming and update of original design located at: https://github.com/UniversalScientificTechnologies/AIRDOSC01/tree/a4267a465eca13d7ddbf4bbd4efce818695a9dc9/hw/sch_pcb/AIRDOSC01A_PCB01C/hw/sch_pcb
Other:
- title: NAME -> SIPM02C
